File: active-diff.kicad_pcb (KiCad board)
At the start: 2 copper layers, 107.6 x 20 mm, 84 parts, among them J1 INPUT-, J2 USB-C, J3 JST-PH-2, J4 INPUT+, J5 BNC, J6 JST-PH-2, Q1 FS8205A, SW1 SLIDE_SWITCH, U1 AD8130, U2 DW01A, U3 TPS61220, U5 TPS60403, U6 ADP7142AUJZ-5.0, U7 MCP73831T, U8 ADP7182-5.0

Commit message: R1 sent to JLCPCB
Parts:
- removed the REF** at (99.9, 120.2)
- added ?: , , F.Cu at (91.2, 120.0)
- added R16: 5M1, Resistor_SMD:R_0603_1608Metric_Pad0.98x0.95mm_HandSolder, F.Cu at (92.3, 114.8)
- added R7: 5M1, Resistor_SMD:R_0603_1608Metric_Pad0.98x0.95mm_HandSolder, F.Cu at (92.3, 125.2)
- added REF**: ToolingHole_1.152mm, MountingHole:ToolingHole_1.152mm, F.Cu at (99.9, 120.0)
- R1, R4: value 9M -> 3M9
- moved C5 0.20 mm to (95.2, 123.0)
- moved J4 0.20 mm to (87.6, 123.0)
- moved TP3 0.20 mm to (91.2, 123.0)
Connections:
- R1 pad 1: /Input Attenuator1/In -> Net-(R1-Pad1)
- R4 pad 1: /Input Attenuator/In -> Net-(R4-Pad1)
Routing:
- net /Input Attenuator/In: track 10.2 -> 7.32 mm
- net /Input Attenuator1/In: track 10.2 -> 7.33 mm
- net Net-(R4-Pad1): track 0.00 -> 2.54 mm
- net Net-(R1-Pad1): track 0.00 -> 2.09 mm
Other:
- board text added: "2026-02-05"
- board text added: "Active differential Probe, Rev1"
- board text added: "P"
