File: DiffAmp.kicad_sch (KiCad schematic)
At the start: 8 parts, among them U1 AD8130

Commit message: Update documentation and schematics for AD8130 design
Documentation updates:
- CLAUDE.md: Fixed schematic hierarchy (removed buffer.kicad_sch,
  updated DiffAmp description to AD8130, corrected bandwidth to 270MHz)
- Power supply design doc: Updated load requirements for AD8130
  (single IC vs 3 ICs), corrected circuit block references

Schematic updates:
- Renamed JLCPCB# property to JLCPCB Part# in all schematic files
  (InputAttenuator, DiffAmp, Power, active-diff)
- Removed unused buffer.kicad_sch (orphaned from earlier design)

New files:
- docs/index.html: Documentation index with categories
  (Design Input, Component Selection, Datasheets, Calibration,
  Manufacturing, KiCad Project)

Co-Authored-By: Claude Opus 4.5 <noreply@anthropic.com>
Parts:
- C3, C9: JLCPCB Part# (none) -> C60474; JLCPCB# C60474 -> (none)
- R6: JLCPCB Part# (none) -> C25744; JLCPCB# C25744 -> (none)
- RF2: JLCPCB Part# (none) -> C11702; JLCPCB# C11702 -> (none)
- U1: JLCPCB Part# (none) -> C41661; JLCPCB# C41661 -> (none)
Changed lines of the file:
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@@
 			)
 		)
-		(property "JLCPCB#" ""
+		(property "JLCPCB Part#" ""
 			(at 116.84 78.74 0)
 			(effects
@@
 			)
 		)
-		(property "JLCPCB#" "C25744"
+		(property "JLCPCB Part#" "C25744"
 			(at 124.46 82.55 90)
 			(effects
@@
 			)
 		)
-		(property "JLCPCB#" "C60474"
+		(property "JLCPCB Part#" "C60474"
 			(at 128.27 133.35 0)
 			(effects
@@
 			)
 		)
-		(property "JLCPCB#" "C60474"
+		(property "JLCPCB Part#" "C60474"
 			(at 140.97 133.35 0)
 			(effects
@@
 			)
 		)
-		(property "JLCPCB#" "C11702"
+		(property "JLCPCB Part#" "C11702"
 			(at 153.67 96.52 90)
 			(effects
@@
 			)
 		)
-		(property "JLCPCB#" ""
+		(property "JLCPCB Part#" ""
 			(at 156.21 93.98 0)
 			(effects
@@
 			)
 		)
-		(property "JLCPCB#" "C41661"
+		(property "JLCPCB Part#" "C41661"
 			(at 132.08 93.98 0)
 			(effects
@@
 			)
 		)
-		(property "JLCPCB#" ""
+		(property "JLCPCB Part#" ""
 			(at 144.78 101.6 90)
 			(effects
