File: InputAttenuator.kicad_sch (KiCad schematic)
At the start: 8 parts

Commit message: Update documentation and schematics for AD8130 design
Documentation updates:
- CLAUDE.md: Fixed schematic hierarchy (removed buffer.kicad_sch,
  updated DiffAmp description to AD8130, corrected bandwidth to 270MHz)
- Power supply design doc: Updated load requirements for AD8130
  (single IC vs 3 ICs), corrected circuit block references

Schematic updates:
- Renamed JLCPCB# property to JLCPCB Part# in all schematic files
  (InputAttenuator, DiffAmp, Power, active-diff)
- Removed unused buffer.kicad_sch (orphaned from earlier design)

New files:
- docs/index.html: Documentation index with categories
  (Design Input, Component Selection, Datasheets, Calibration,
  Manufacturing, KiCad Project)

Co-Authored-By: Claude Opus 4.5 <noreply@anthropic.com>
Parts:
- C5, C6: JLCPCB Part# (none) -> C22468120; JLCPCB# C22468120 -> (none)
- D1: JLCPCB Part# (none) -> C2827694; JLCPCB# C2827694 -> (none)
- R4: JLCPCB Part# (none) -> C423039; JLCPCB# C423039 -> (none)
- R5: JLCPCB Part# (none) -> C4165581; JLCPCB# C4165581 -> (none)
- R7: JLCPCB Part# (none) -> C13320; JLCPCB# C13320 -> (none)
Changed lines of the file:
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@@
 			)
 		)
-		(property "JLCPCB#" ""
+		(property "JLCPCB Part#" ""
 			(at 102.87 86.36 0)
 			(effects
@@
 			)
 		)
-		(property "JLCPCB#" "C2827694"
+		(property "JLCPCB Part#" "C2827694"
 			(at 167.64 97.79 90)
 			(effects
@@
 			)
 		)
-		(property "JLCPCB#" "C22468120"
+		(property "JLCPCB Part#" "C22468120"
 			(at 121.92 97.79 90)
 			(effects
@@
 			)
 		)
-		(property "JLCPCB#" "C423039"
+		(property "JLCPCB Part#" "C423039"
 			(at 121.92 90.17 90)
 			(effects
@@
 			)
 		)
-		(property "JLCPCB#" "C22468120"
+		(property "JLCPCB Part#" "C22468120"
 			(at 143.51 107.95 0)
 			(effects
@@
 			)
 		)
-		(property "JLCPCB#" "C4165581"
+		(property "JLCPCB Part#" "C4165581"
 			(at 137.16 107.95 0)
 			(effects
@@
 			)
 		)
-		(property "JLCPCB#" "C13320"
+		(property "JLCPCB Part#" "C13320"
 			(at 110.49 90.17 90)
 			(effects
@@
 			)
 		)
-		(property "JLCPCB#" ""
+		(property "JLCPCB Part#" ""
 			(at 179.07 90.17 0)
 			(effects
