File: Power.kicad_sch (KiCad schematic)
At the start: 52 parts, among them J2 USB-C, J3 JST-PH-2, J6 JST-PH-2, Q1 FS8205A, SW1 SLIDE_SWITCH, U2 DW01A, U3 TPS61220, U5 TPS60403, U6 ADP7142AUJZ-5.0, U7 MCP73831T, U8 ADP7182-5.0

Commit message: Update documentation and schematics for AD8130 design
Documentation updates:
- CLAUDE.md: Fixed schematic hierarchy (removed buffer.kicad_sch,
  updated DiffAmp description to AD8130, corrected bandwidth to 270MHz)
- Power supply design doc: Updated load requirements for AD8130
  (single IC vs 3 ICs), corrected circuit block references

Schematic updates:
- Renamed JLCPCB# property to JLCPCB Part# in all schematic files
  (InputAttenuator, DiffAmp, Power, active-diff)
- Removed unused buffer.kicad_sch (orphaned from earlier design)

New files:
- docs/index.html: Documentation index with categories
  (Design Input, Component Selection, Datasheets, Calibration,
  Manufacturing, KiCad Project)

Co-Authored-By: Claude Opus 4.5 <noreply@anthropic.com>
Parts:
- C11, C13, C14, C17, C8: JLCPCB Part# (none) -> C59782; JLCPCB# C59782 -> (none)
- C12, C16, C22, C23: JLCPCB Part# (none) -> C237435; JLCPCB# C237435 -> (none)
- C15, C18, C19, C7: JLCPCB Part# (none) -> C60474; JLCPCB# C60474 -> (none)
- C20: JLCPCB Part# (none) -> C15195; JLCPCB# C15195 -> (none)
- C21: JLCPCB Part# (none) -> C296720; JLCPCB# C296720 -> (none)
- D3, D5: JLCPCB Part# (none) -> C2135; JLCPCB# C2135 -> (none)
- D4: JLCPCB Part# (none) -> C2295; JLCPCB# C2295 -> (none)
- D6: JLCPCB Part# (none) -> C2297; JLCPCB# C2297 -> (none)
- J2: JLCPCB Part# (none) -> C165948; JLCPCB# C165948 -> (none)
- J3, J6: JLCPCB Part# (none) -> C173752; JLCPCB# C173752 -> (none)
- L1: JLCPCB Part# (none) -> C136233; JLCPCB# C136233 -> (none)
- Q1: JLCPCB Part# (none) -> C2830320; JLCPCB# C2830320 -> (none)
- R10: JLCPCB Part# (none) -> C25741; JLCPCB# C25741 -> (none)
- R11: JLCPCB Part# (none) -> C26083; JLCPCB# C26083 -> (none)
- R12, R13: JLCPCB Part# (none) -> C25905; JLCPCB# C25905 -> (none)
- R14, R3, R9: JLCPCB Part# (none) -> C11702; JLCPCB# C11702 -> (none)
- R15: JLCPCB Part# (none) -> C4109; JLCPCB# C4109 -> (none)
- R8: JLCPCB Part# (none) -> C25077; JLCPCB# C25077 -> (none)
- SW1: JLCPCB Part# (none) -> C221841; JLCPCB# C221841 -> (none)
- U2: JLCPCB Part# (none) -> C2927799; JLCPCB# C2927799 -> (none)
- U3: JLCPCB Part# (none) -> C15421; JLCPCB# C15421 -> (none)
- U5: JLCPCB Part# (none) -> C11338; JLCPCB# C11338 -> (none)
- U6: JLCPCB Part# (none) -> C659367; JLCPCB# C659367 -> (none)
- U7: JLCPCB Part# (none) -> C424093; JLCPCB# C424093 -> (none)
- U8: JLCPCB Part# (none) -> C514357; JLCPCB# C514357 -> (none)
Changed lines of the file:
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@@
 			)
 		)
-		(property "JLCPCB#" "C2135"
+		(property "JLCPCB Part#" "C2135"
 			(at 67.31 27.94 90)
 			(effects
@@
 			)
 		)
-		(property "JLCPCB#" "C296720"
+		(property "JLCPCB Part#" "C296720"
 			(at 250.19 43.18 0)
 			(effects
@@
 			)
 		)
-		(property "JLCPCB#" "C2135"
+		(property "JLCPCB Part#" "C2135"
 			(at 341.63 50.8 90)
 			(effects
@@
 			)
 		)
-		(property "JLCPCB#" "C15195"
+		(property "JLCPCB Part#" "C15195"
 			(at 179.07 184.15 0)
 			(effects
@@
 			)
 		)
-		(property "JLCPCB#" "C60474"
+		(property "JLCPCB Part#" "C60474"
 			(at 166.37 184.15 0)
 			(effects
@@
 			)
 		)
-		(property "JLCPCB#" ""
+		(property "JLCPCB Part#" ""
 			(at 77.47 175.26 0)
 			(effects
@@
 			)
 		)
-		(property "JLCPCB#" "C237435"
+		(property "JLCPCB Part#" "C237435"
 			(at 325.12 44.45 0)
 			(effects
@@
 			)
 		)
-		(property "JLCPCB#" ""
+		(property "JLCPCB Part#" ""
 			(at 156.21 109.22 0)
 			(effects
@@
 			)
 		)
-		(property "JLCPCB#" "C25905 "
+		(property "JLCPCB Part#" "C25905 "
 			(at 88.9 64.77 0)
 			(effects
@@
 			)
 		)
-		(property "JLCPCB#" "C25741"
+		(property "JLCPCB Part#" "C25741"
 			(at 316.23 52.07 0)
 			(effects
@@
 			)
 		)
-		(property "JLCPCB#" "C11702"
+		(property "JLCPCB Part#" "C11702"
 			(at 212.09 60.96 90)
 			(effects
@@
 			)
 		)
-		(property "JLCPCB#" "C11702"
+		(property "JLCPCB Part#" "C11702"
 			(at 369.57 58.42 0)
 			(effects
@@
 			)
 		)
-		(property "JLCPCB#" ""
+		(property "JLCPCB Part#" ""
 			(at 139.7 40.64 0)
 			(effects
@@
 			)
 		)
-		(property "JLCPCB#" "C514357"
+		(property "JLCPCB Part#" "C514357"
 			(at 134.62 182.88 0)
 			(effects
@@
 			)
 		)
-		(property "JLCPCB#" "C221841"
+		(property "JLCPCB Part#" "C221841"
 			(at 358.14 50.8 0)
 			(effects
@@
 			)
 		)
-		(property "JLCPCB#" "C136233"
+		(property "JLCPCB Part#" "C136233"
 			(at 298.45 25.4 90)
 			(effects
@@
 			)
 		)
-		(property "JLCPCB#" "C173752 "
+		(property "JLCPCB Part#" "C173752 "
 			(at 320.04 74.93 0)
 			(effects
@@
 			)
 		)
-		(property "JLCPCB#" "C25905 "
+		(property "JLCPCB Part#" "C25905 "
 			(at 97.79 64.77 0)
 			(effects
@@
 			)
 		)
-		(property "JLCPCB#" "C165948"
+		(property "JLCPCB Part#" "C165948"
 			(at 46.99 50.8 0)
 			(effects
@@
 			)
 		)
-		(property "JLCPCB#" "C15421"
+		(property "JLCPCB Part#" "C15421"
 			(at 298.45 39.37 0)
 			(effects
@@
 			)
 		)
-		(property "JLCPCB#" ""
+		(property "JLCPCB Part#" ""
 			(at 383.54 50.8 0)
 			(effects
@@
 			)
 		)
-		(property "JLCPCB#" ""
+		(property "JLCPCB Part#" ""
 			(at 172.72 41.91 0)
 			(effects
@@
 			)
 		)
-		(property "JLCPCB#" ""
+		(property "JLCPCB Part#" ""
 			(at 168.91 109.22 0)
 			(effects
@@
 			)
 		)
-		(property "JLCPCB#" "C11338"
+		(property "JLCPCB Part#" "C11338"
 			(at 58.42 186.69 0)
 			(effects
@@
 			)
 		)
-		(property "JLCPCB#" ""
+		(property "JLCPCB Part#" ""
 			(at 172.72 175.26 0)
 			(effects
@@
 			)
 		)
-		(property "JLCPCB#" "C60474"
+		(property "JLCPCB Part#" "C60474"
 			(at 175.26 59.69 0)
 			(effects
@@
 			)
 		)
-		(property "JLCPCB#" ""
+		(property "JLCPCB Part#" ""
 			(at 349.25 50.8 0)
 			(effects
@@
 			)
 		)
-		(property "JLCPCB#" "C173752 "
+		(property "JLCPCB Part#" "C173752 "
 			(at 158.75 25.4 90)
 			(effects
@@
 			)
 		)
-		(property "JLCPCB#" "C60474"
+		(property "JLCPCB Part#" "C60474"
 			(at 59.69 123.19 0)
 			(effects
@@
 			)
 		)
-		(property "JLCPCB#" "C2830320"
+		(property "JLCPCB Part#" "C2830320"
 			(at 219.71 41.91 0)
 			(effects
@@
 			)
 		)
-		(property "JLCPCB#" "C2830320"
+		(property "JLCPCB Part#" "C2830320"
 			(at 205.74 41.91 0)
 			(effects
@@
 			)
 		)
-		(property "JLCPCB#" "C237435"
+		(property "JLCPCB Part#" "C237435"
 			(at 154.94 184.15 0)
 			(effects
@@
 			)
 		)
-		(property "JLCPCB#" "C237435"
+		(property "JLCPCB Part#" "C237435"
 			(at 107.95 119.38 0)
 			(effects
@@
 			)
 		)
-		(property "JLCPCB#" "C2295"
+		(property "JLCPCB Part#" "C2295"
 			(at 123.19 26.67 0)
 			(effects
@@
 			)
 		)
-		(property "JLCPCB#" "C4109"
+		(property "JLCPCB Part#" "C4109"
 			(at 127 52.07 0)
 			(effects
@@
 			)
 		)
-		(property "JLCPCB#" "C11702"
+		(property "JLCPCB Part#" "C11702"
 			(at 100.33 26.67 90)
 			(effects
@@
 			)
 		)
-		(property "JLCPCB#" "C237435"
+		(property "JLCPCB Part#" "C237435"
 			(at 262.89 43.18 0)
 			(effects
@@
 			)
 		)
-		(property "JLCPCB#" "C59782"
+		(property "JLCPCB Part#" "C59782"
 			(at 31.75 193.04 0)
 			(effects
@@
 			)
 		)
-		(property "JLCPCB#" "C25077"
+		(property "JLCPCB Part#" "C25077"
 			(at 168.91 50.8 90)
 			(effects
@@
 			)
 		)
-		(property "JLCPCB#" ""
+		(property "JLCPCB Part#" ""
 			(at 336.55 74.93 0)
 			(effects
@@
 			)
 		)
-		(property "JLCPCB#" ""
+		(property "JLCPCB Part#" ""
 			(at 85.09 26.67 0)
 			(effects
@@
 			)
 		)
-		(property "JLCPCB#" ""
+		(property "JLCPCB Part#" ""
 			(at 162.56 109.22 0)
 			(effects
@@
 			)
 		)
-		(property "JLCPCB#" "C26083"
+		(property "JLCPCB Part#" "C26083"
 			(at 316.23 41.91 0)
 			(effects
@@
 			)
 		)
-		(property "JLCPCB#" ""
+		(property "JLCPCB Part#" ""
 			(at 341.63 36.83 0)
 			(effects
@@
 			)
 		)
-		(property "JLCPCB#" "C659367"
+		(property "JLCPCB Part#" "C659367"
 			(at 82.55 120.65 0)
 			(effects
@@
 			)
 		)
-		(property "JLCPCB#" "C59782"
+		(property "JLCPCB Part#" "C59782"
 			(at 58.42 172.72 90)
 			(effects
@@
 			)
 		)
-		(property "JLCPCB#" "C59782"
+		(property "JLCPCB Part#" "C59782"
 			(at 45.72 123.19 0)
 			(effects
@@
 			)
 		)
-		(property "JLCPCB#" "C59782"
+		(property "JLCPCB Part#" "C59782"
 			(at 114.3 187.96 0)
 			(effects
@@
 			)
 		)
-		(property "JLCPCB#" "C2297"
+		(property "JLCPCB Part#" "C2297"
 			(at 369.57 66.04 90)
 			(effects
@@
 			)
 		)
-		(property "JLCPCB#" "C60474"
+		(property "JLCPCB Part#" "C60474"
 			(at 119.38 119.38 0)
 			(effects
@@
 			)
 		)
-		(property "JLCPCB#" "C2927799"
+		(property "JLCPCB Part#" "C2927799"
 			(at 187.96 55.88 0)
 			(effects
@@
 			)
 		)
-		(property "JLCPCB#" "C424093"
+		(property "JLCPCB Part#" "C424093"
 			(at 109.22 38.1 0)
 			(effects
@@
 			)
 		)
-		(property "JLCPCB#" "C59782"
+		(property "JLCPCB Part#" "C59782"
 			(at 77.47 191.77 0)
 			(effects
