File: active-diff.kicad_sch (KiCad schematic)
At the start: 8 parts, among them J1 INPUT-, J4 INPUT+, J5 BNC

Commit message: Update documentation and schematics for AD8130 design
Documentation updates:
- CLAUDE.md: Fixed schematic hierarchy (removed buffer.kicad_sch,
  updated DiffAmp description to AD8130, corrected bandwidth to 270MHz)
- Power supply design doc: Updated load requirements for AD8130
  (single IC vs 3 ICs), corrected circuit block references

Schematic updates:
- Renamed JLCPCB# property to JLCPCB Part# in all schematic files
  (InputAttenuator, DiffAmp, Power, active-diff)
- Removed unused buffer.kicad_sch (orphaned from earlier design)

New files:
- docs/index.html: Documentation index with categories
  (Design Input, Component Selection, Datasheets, Calibration,
  Manufacturing, KiCad Project)

Co-Authored-By: Claude Opus 4.5 <noreply@anthropic.com>
Parts:
- ROUT1: JLCPCB Part# (none) -> C227387; JLCPCB# C227387 -> (none)
- ROUT2: JLCPCB Part# (none) -> C17168; JLCPCB# C17168 -> (none)
Changed lines of the file:
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@@
 			)
 		)
-		(property "JLCPCB#" ""
+		(property "JLCPCB Part#" ""
 			(at 36.83 60.96 0)
 			(effects
@@
 			)
 		)
-		(property "JLCPCB#" ""
+		(property "JLCPCB Part#" ""
 			(at 255.27 77.47 0)
 			(effects
@@
 			)
 		)
-		(property "JLCPCB#" ""
+		(property "JLCPCB Part#" ""
 			(at 232.41 92.71 0)
 			(effects
@@
 			)
 		)
-		(property "JLCPCB#" "C17168"
+		(property "JLCPCB Part#" "C17168"
 			(at 227.33 77.47 90)
 			(effects
@@
 			)
 		)
-		(property "JLCPCB#" ""
+		(property "JLCPCB Part#" ""
 			(at 219.71 72.39 0)
 			(effects
@@
 			)
 		)
-		(property "JLCPCB#" "C227387"
+		(property "JLCPCB Part#" "C227387"
 			(at 212.09 77.47 90)
 			(effects
@@
 			)
 		)
-		(property "JLCPCB#" ""
+		(property "JLCPCB Part#" ""
 			(at 36.83 106.68 0)
 			(effects
@@
 			)
 		)
-		(property "JLCPCB#" ""
+		(property "JLCPCB Part#" ""
 			(at 246.38 72.39 0)
 			(effects
